Commit message: updates

File: src/ur5e_motion_controller/my_urdf/ur_ur5e_fake_berry.xacro (robot description, xacro)
@@ -7,7 +7,7 @@
     <link name="blackberry">
         <visual>
-        <origin xyz="0 0 0" rpy="0 0 0"/>
+        <origin xyz="0 0 -0.07748" rpy="0 0 0"/>
         <geometry>
-            <mesh filename="file://$(find ur5e_motion_controller)/meshes/fake_berry.stl" scale="0.001 0.001 0.001"/>
+            <mesh filename="file://$(find ur5e_motion_controller)/meshes/fake_berry_2.stl" scale="0.001 0.001 0.001"/>
         </geometry>
         <material name="">
@@ -19,5 +19,5 @@
         <parent link="tool0"/>
         <child link="blackberry"/>
-        <origin xyz="0 0 0.1" rpy="0 0 0"/>
+        <origin xyz="0 0 0.07748" rpy="0 0 0"/>
     </joint>
       </xacro:macro>
