Commit message: update

File: src/ur5e_motion_controller/my_urdf/my_ur5e_robot.xacro (robot description, xacro)
@@ -3,5 +3,5 @@
   <!-- Include the standard UR5e robot -->
   <xacro:include filename="$(find ur_description)/urdf/ur.urdf.xacro"/>
-  <!-- <xacro:ur_robot ur_type="ur5e" prefix=""/> -->
+  <!-- <xacro:ur_robot ur_type="ur5e" prefix=""/>  -->
   <!-- Include the blackberry macro-->
   <xacro:include filename="$(find ur5e_motion_controller)/my_urdf/ur_ur5e_fake_berry.xacro"/>

File: src/ur5e_motion_controller/my_urdf/ur_ur5e_fake_berry.xacro (robot description, xacro)
@@ -3,14 +3,12 @@
   <xacro:macro name="add_blackberry" params="">
     <!-- Define blackberry link -->
-    <!-- Gray: 0.2 0.2 0.2 1 -->
-    <!-- Red: 1 0 0 1 -->
     <link name="blackberry">
         <visual>
-        <origin xyz="0 0 -0.07748" rpy="0 0 0"/>
+        <origin xyz="0.0 0.0 -0.07748" rpy="0.0 0.0 0.0"/>
         <geometry>
             <mesh filename="file://$(find ur5e_motion_controller)/meshes/fake_berry_2.stl" scale="0.001 0.001 0.001"/>
         </geometry>
         <material name="">
-            <color rgba="1.0 0.0. 0.0 1.0 "/>
+            <color rgba="1.0 0.0 0.0 1.0 "/> <!-- Red: 1 0 0 1 --> <!-- Gray: 0.2 0.2 0.2 1 -->
         </material>
         </visual>
@@ -19,6 +17,6 @@
         <parent link="tool0"/>
         <child link="blackberry"/>
-        <origin xyz="0 0 0.07748" rpy="0 0 0"/>
+        <origin xyz="0.0 0.0 0.07748" rpy="0.0 0.0 0.0"/>
     </joint>
-      </xacro:macro>
+    </xacro:macro>
 </robot>
