Commit message: fixed collision ref frame

File: src/ur5e_motion_controller/urdf/ur5e_berry.xacro (robot description, xacro)
@@ -13,6 +13,7 @@
         physical_parameters_file="$(find ur_description)/config/ur5e/physical_parameters.yaml"
         visual_parameters_file="$(find ur_description)/config/ur5e/visual_parameters.yaml"
+        initial_positions="${dict(shoulder_pan_joint=-1.57,shoulder_lift_joint=-1.57,elbow_joint=-1.70,wrist_1_joint=-1.57,wrist_2_joint=-1.57,wrist_3_joint=0.0)}"
     >
-        <origin xyz="0 0 0" rpy="0 0 0" />
+        <origin xyz="0 0 1.79" rpy="${pi} 0 ${pi}" />
     </xacro:ur_robot>
     <link name="blackberry">

File: src/ur5e_motion_controller/urdf/ur5e_berry_control.xacro (robot description, xacro)
@@ -69,4 +69,5 @@
         fake_sensor_commands="$(arg fake_sensor_commands)"
         headless_mode="$(arg headless_mode)"
+        initial_positions="${dict(shoulder_pan_joint=-1.57,shoulder_lift_joint=-1.57,elbow_joint=-1.70,wrist_1_joint=-1.57,wrist_2_joint=-1.57,wrist_3_joint=0.0)}"
     />
     <!--Create
